Commit message: Update URDF for mycobot_280_arduino: adjust mesh scales and formatting

File: mycobot_description/urdf/mycobot_280_arduino/mycobot_280_arduino.urdf (robot description, URDF)
Before this commit: robot firefighter, 8 links, 7 joints
Links:
- link g_base: geometry collision mesh filename=package://mycobot_description/urdf/mycobot_280_arduino/G_ba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 scale=0.001 0.001 0.001; visual mesh filename=package://mycobot_description/urdf/mycobot_280_arduino/G_ba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 scale=0.001 0.001 0.001
- link joint1: geometry collision mesh filename=package://mycobot_description/urdf/mycobot_280_arduino/join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 scale=0.001 0.001 0.001; visual mesh filename=package://mycobot_description/urdf/mycobot_280_arduino/join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 scale=0.001 0.001 0.001

Commit message: Update URDF origin for joint6 (rotate 45 deg)

File: mycobot_description/urdf/mycobot_280_arduino/mycobot_280_arduino.urdf (robot description, URDF)
Before this commit: robot mycobot_280_arduino, 8 links, 7 joints
Joints:
- joint joint6output_to_joint6: origin xyz=0 0.0456 0 rpy=-1.5708 0 0 -> xyz=0 0.0456 0 rpy=-1.5708 0.7854 0

Commit message: Update effort and velocity limits in mycobot_280_arduino.urdf

File: mycobot_description/urdf/mycobot_280_arduino/mycobot_280_arduino.urdf (robot description, URDF)
Before this commit: robot mycobot_280_arduino, 8 links, 7 joints
Joints:
- joint g_base_to_joint1: limit lower=-3.14 upper=3.14159 effort=1000.0 velocity=0 -> lower=-3.14 upper=3.14159 effort=1.0 velocity=2.6
- joint joint2_to_joint1: limit lower=-2.9321 upper=2.9321 effort=1000.0 velocity=0 -> lower=-2.9321 upper=2.9321 effort=1.0 velocity=2.6
- joint joint3_to_joint2: limit lower=-2.3561 upper=2.3561 effort=1000.0 velocity=0 -> lower=-2.3561 upper=2.3561 effort=1.0 velocity=2.6
- joint joint4_to_joint3: limit lower=-2.6179 upper=2.6179 effort=1000.0 velocity=0 -> lower=-2.6179 upper=2.6179 effort=1.0 velocity=2.6
- joint joint5_to_joint4: limit lower=-2.5307 upper=2.5307 effort=1000.0 velocity=0 -> lower=-2.5307 upper=2.5307 effort=1.0 velocity=2.6
- joint joint6_to_joint5: limit lower=-2.8797 upper=2.8797 effort=1000.0 velocity=0 -> lower=-2.8797 upper=2.8797 effort=1.0 velocity=2.6
- joint joint6output_to_joint6: limit lower=-3.14 upper=3.14159 effort=1000.0 velocity=0 -> lower=-3.14 upper=3.14159 effort=1.0 velocity=2.6
