Commit message: Stock protocol reference, official firmware sources, servo types and measured joint limits

File: mycobot_description/urdf/mycobot_280_arduino/mycobot_280_arduino.urdf (robot description, URDF)
Before this commit: robot mycobot_280_arduino, 8 links, 7 joints
Joints:
- joint joint2_to_joint1: limit lower=-2.9321 upper=2.9321 effort=1.0 velocity=2.6 -> lower=-2.8798 upper=2.8798 effort=1.0 velocity=2.6
- joint joint3_to_joint2: limit lower=-2.3561 upper=2.3561 effort=1.0 velocity=2.6 -> lower=-2.4435 upper=2.4435 effort=1.0 velocity=2.6
- joint joint4_to_joint3: limit lower=-2.6179 upper=2.6179 effort=1.0 velocity=2.6 -> lower=-2.6180 upper=2.6180 effort=1.0 velocity=2.6
- joint joint5_to_joint4: limit lower=-2.5307 upper=2.5307 effort=1.0 velocity=2.6 -> lower=-2.6180 upper=2.6180 effort=1.0 velocity=2.6
- joint joint6_to_joint5: limit lower=-2.8797 upper=2.8797 effort=1.0 velocity=2.6 -> lower=-2.7925 upper=2.7925 effort=1.0 velocity=2.6

Commit message: Robot description: one source (URDF xacro, ros2_control joint_limits.yaml, servos.yaml) and tools/gen_robot.py for the URDFs and the firmware, Control page, simulator and Julia tables

File: mycobot_description/urdf/mycobot_280_arduino/mycobot_280_arduino.urdf (robot description, URDF)
Before this commit: robot mycobot_280_arduino, 8 links, 7 joints
Joints:
- joint g_base_to_joint1: axis 0 0 0 -> (none); limit lower=-3.14 upper=3.14159 effort=1.0 velocity=2.6 -> (none)
- joint joint2_to_joint1: limit lower=-2.8798 upper=2.8798 effort=1.0 velocity=2.6 -> lower=-2.879793 upper=2.879793 effort=0.0 velocity=1.570796
- joint joint3_to_joint2: limit lower=-2.4435 upper=2.4435 effort=1.0 velocity=2.6 -> lower=-2.443461 upper=2.443461 effort=0.0 velocity=1.570796; origin xyz=0 0  0 rpy=0 1.5708 -1.5708 -> xyz=0 0 0 rpy=0 1.5708 -1.5708
- joint joint4_to_joint3: axis  0 0 1 -> 0 0 1; limit lower=-2.6180 upper=2.6180 effort=1.0 velocity=2.6 -> lower=-2.617994 upper=2.617994 effort=0.0 velocity=1.570796; origin xyz=  -0.1104 0 0    rpy=0 0 0 -> xyz=-0.1104 0 0 rpy=0 0 0
- joint joint5_to_joint4: axis  0 0 1 -> 0 0 1; limit lower=-2.6180 upper=2.6180 effort=1.0 velocity=2.6 -> lower=-2.617994 upper=2.617994 effort=0.0 velocity=1.570796
- joint joint6_to_joint5: limit lower=-2.7925 upper=2.7925 effort=1.0 velocity=2.6 -> lower=-2.792527 upper=2.792527 effort=0.0 velocity=1.570796
- joint joint6output_to_joint6: limit lower=-3.14 upper=3.14159 effort=1.0 velocity=2.6 -> lower=-3.141593 upper=3.141593 effort=0.0 velocity=1.570796

File: website/public/robot/mycobot_280_arduino.urdf (robot description, URDF)
Before this commit: robot mycobot_280_arduino, 8 links, 7 joints
Joints:
- joint g_base_to_joint1: axis 0 0 0 -> (none); limit lower=-3.14 upper=3.14159 effort=1.0 velocity=2.6 -> (none)
- joint joint2_to_joint1: limit lower=-2.8798 upper=2.8798 effort=1.0 velocity=2.6 -> lower=-2.879793 upper=2.879793 effort=0.0 velocity=1.570796
- joint joint3_to_joint2: limit lower=-2.4435 upper=2.4435 effort=1.0 velocity=2.6 -> lower=-2.443461 upper=2.443461 effort=0.0 velocity=1.570796
- joint joint4_to_joint3: limit lower=-2.6180 upper=2.6180 effort=1.0 velocity=2.6 -> lower=-2.617994 upper=2.617994 effort=0.0 velocity=1.570796
- joint joint5_to_joint4: limit lower=-2.6180 upper=2.6180 effort=1.0 velocity=2.6 -> lower=-2.617994 upper=2.617994 effort=0.0 velocity=1.570796
- joint joint6_to_joint5: limit lower=-2.7925 upper=2.7925 effort=1.0 velocity=2.6 -> lower=-2.792527 upper=2.792527 effort=0.0 velocity=1.570796
- joint joint6output_to_joint6: limit lower=-3.14 upper=3.14159 effort=1.0 velocity=2.6 -> lower=-3.141593 upper=3.141593 effort=0.0 velocity=1.570796

Commit message: Controller firmware 4.4.1: J6 limit ±135° with the gripper on (its cable stops J6 at −237.1° and +139.9°); gripper mount at 45° recorded

File: mycobot_description/urdf/mycobot_280_arduino/mycobot_280_arduino.urdf (robot description, URDF)
Before this commit: robot mycobot_280_arduino, 8 links, 7 joints
Joints:
- joint joint6output_to_joint6: limit lower=-3.141593 upper=3.141593 effort=0.0 velocity=1.570796 -> lower=-2.356194 upper=2.356194 effort=0.0 velocity=1.570796

File: website/public/robot/mycobot_280_arduino.urdf (robot description, URDF)
Before this commit: robot mycobot_280_arduino, 8 links, 7 joints
Joints:
- joint joint6output_to_joint6: limit lower=-3.141593 upper=3.141593 effort=0.0 velocity=1.570796 -> lower=-2.356194 upper=2.356194 effort=0.0 velocity=1.570796

Commit message: Controller firmware 4.5.0: J6 multi-turn (phase bit 4 and angle limits 0/0 at power-up, the turn from the power-up reading; tested to −231.8° by hand and −209.3° under control), non-symmetric limits, J6 −220° to +135°

File: mycobot_description/urdf/mycobot_280_arduino/mycobot_280_arduino.urdf (robot description, URDF)
Before this commit: robot mycobot_280_arduino, 8 links, 7 joints
Joints:
- joint joint6output_to_joint6: limit lower=-2.356194 upper=2.356194 effort=0.0 velocity=1.570796 -> lower=-3.839724 upper=2.356194 effort=0.0 velocity=1.570796

File: website/public/robot/mycobot_280_arduino.urdf (robot description, URDF)
Before this commit: robot mycobot_280_arduino, 8 links, 7 joints
Joints:
- joint joint6output_to_joint6: limit lower=-2.356194 upper=2.356194 effort=0.0 velocity=1.570796 -> lower=-3.839724 upper=2.356194 effort=0.0 velocity=1.570796

Commit message: Controller firmware 4.5.1: J6 limits −225° to +135° (one full turn of the gripper), power-up guard when the J6 turn is not known

File: mycobot_description/urdf/mycobot_280_arduino/mycobot_280_arduino.urdf (robot description, URDF)
Before this commit: robot mycobot_280_arduino, 8 links, 7 joints
Joints:
- joint joint6output_to_joint6: limit lower=-3.839724 upper=2.356194 effort=0.0 velocity=1.570796 -> lower=-3.926991 upper=2.356194 effort=0.0 velocity=1.570796

File: website/public/robot/mycobot_280_arduino.urdf (robot description, URDF)
Before this commit: robot mycobot_280_arduino, 8 links, 7 joints
Joints:
- joint joint6output_to_joint6: limit lower=-3.839724 upper=2.356194 effort=0.0 velocity=1.570796 -> lower=-3.926991 upper=2.356194 effort=0.0 velocity=1.570796

Commit message: Gripper body 2.4 mm nearer J6 (the flange face: 43.2 mm, was 45.6) and 1.2 mm to the side, and new joint zero offsets, from the palm holes and the arm outline in 55 camera snapshots (held-out palm holes 10.0 -> 2.7 px)

File: mycobot_description/urdf/mycobot_280_arduino/mycobot_280_arduino.urdf (robot description, URDF)
Before this commit: robot mycobot_280_arduino, 8 links, 7 joints
Joints:
- joint joint6output_to_joint6: origin xyz=0 0.0456 0 rpy=-1.5708 0.7854 0 -> xyz=0 0.0432 0 rpy=-1.5708 0.7854 0

File: mycobot_description/urdf/mycobot_280_arduino/mycobot_280_arduino.urdf.xacro (robot description, xacro)
@@ -61,5 +61,7 @@
   <xacro:arm_joint name="joint5_to_joint4" parent="joint4" child="joint5" xyz="-0.096 0 0.06462" rpy="0 0 -1.5708" />
   <xacro:arm_joint name="joint6_to_joint5" parent="joint5" child="joint6" xyz="0 -0.07318 0" rpy="1.5708 -1.5708 0" />
-  <xacro:arm_joint name="joint6output_to_joint6" parent="joint6" child="joint6_flange" xyz="0 0.0456 0" rpy="-1.5708 0.7854 0" />
+  <!-- The flange face is 2.4 mm nearer J6 than in Elephant's model (0.0456): the camera puts the gripper body
+       (its palm holes and back-face screws) there, and the body sits on the flange face (2026-10-09). -->
+  <xacro:arm_joint name="joint6output_to_joint6" parent="joint6" child="joint6_flange" xyz="0 0.0432 0" rpy="-1.5708 0.7854 0" />
   <!-- Adaptive gripper (myCobot_gripper_ag), from Elephant's mycobot_280m5_with_gripper_parallel.urdf
        (mycobot_ros; the same meshes and joints as urdf/adaptive_gripper/). Meshes gripper_*.dae are in
@@ -84,9 +86,11 @@
     <xacro:mesh_link name="gripper_right2" mesh="gripper_right2" xyz="-0.005 -0.0195 -0.012" rpy="0 0 0" scale="0.001 0.001 0.001" />
     <xacro:mesh_link name="gripper_right3" mesh="gripper_right3" xyz="-0.012 0.0025 -0.012" rpy="0 0 0" scale="0.001 0.001 0.001" />
-    <!-- The body's back face on the flange, the fingers along the J6 axis. Elephant's roll is 1.579; π/2 here. -->
+    <!-- The body's back face on the flange face, the fingers along the J6 axis. Elephant's roll is 1.579; π/2 here.
+         The camera puts the body 1.2 mm to the side of Elephant's position (flange y; 2026-10-09, the 9 palm holes
+         in 10 snapshots, experiments/kinematic-calib); the flange position is in joint6output_to_joint6. -->
     <joint name="joint6output_to_gripper_base" type="fixed">
       <parent link="joint6_flange" />
       <child link="gripper_base" />
-      <origin xyz="0 0 0.034" rpy="${pi / 2} 0 ${radians(gripper_mount_deg)}" />
+      <origin xyz="-0.0002 0.0012 0.034" rpy="${pi / 2} 0 ${radians(gripper_mount_deg)}" />
     </joint>
     <!-- A finger joint about its z axis. multiplier 0: the actuated joint; otherwise it follows

File: mycobot_description/urdf/mycobot_280_arduino/mycobot_280_arduino_gripper.urdf (robot description, URDF)
Before this commit: robot mycobot_280_arduino, 15 links, 14 joints
Joints:
- joint joint6output_to_gripper_base: origin xyz=0 0 0.034 rpy=1.5707963267948966 0 0.0 -> xyz=-0.0002 0.0012 0.034 rpy=1.5707963267948966 0 0.0
- joint joint6output_to_joint6: origin xyz=0 0.0456 0 rpy=-1.5708 0.7854 0 -> xyz=0 0.0432 0 rpy=-1.5708 0.7854 0

File: website/public/robot/mycobot_280_arduino.urdf (robot description, URDF)
Before this commit: robot mycobot_280_arduino, 8 links, 7 joints
Joints:
- joint joint6output_to_joint6: origin xyz=0 0.0456 0 rpy=-1.5708 0.7854 0 -> xyz=0 0.0432 0 rpy=-1.5708 0.7854 0

File: website/public/robot/mycobot_280_arduino_gripper.urdf (robot description, URDF)
Before this commit: robot mycobot_280_arduino, 15 links, 14 joints
Joints:
- joint joint6output_to_gripper_base: origin xyz=0 0 0.034 rpy=1.5707963267948966 0 0.0 -> xyz=-0.0002 0.0012 0.034 rpy=1.5707963267948966 0 0.0
- joint joint6output_to_joint6: origin xyz=0 0.0456 0 rpy=-1.5708 0.7854 0 -> xyz=0 0.0432 0 rpy=-1.5708 0.7854 0
