Commit message: 3D view: normalize the web URDF number lists (the J3 and J4 axes were NaN, so the links after them vanished)

File: website/public/robot/mycobot_280_arduino.urdf (robot description, URDF)
Before this commit: robot mycobot_280_arduino, 8 links, 7 joints
Joints:
- joint joint3_to_joint2: origin xyz=0 0  0 rpy=0 1.5708 -1.5708 -> xyz=0 0 0 rpy=0 1.5708 -1.5708
- joint joint4_to_joint3: axis  0 0 1 -> 0 0 1; origin xyz=  -0.1104 0 0    rpy=0 0 0 -> xyz=-0.1104 0 0 rpy=0 0 0
- joint joint5_to_joint4: axis  0 0 1 -> 0 0 1
